Commit message: Update for release 2026 (#2081)

File: components/simulations/PicknPlace/robot_config/urdf/ur/ur5/camera.xacro (robot description, xacro)
@@ -64,8 +64,6 @@
       </sensor>
     </link>
-    <!-- Plugin for ROS bridge -->
-    <plugin filename="libgz_ros2_control-system.so" name="gz_ros2_control::GazeboSimROS2ControlPlugin">
-      <parameters>$(find robot_config)/config/camera_bridge.yaml</parameters>
-    </plugin>
+    <!-- ROS bridge no longer needed - camera topics bridged via ros_gz_bridge in launch files -->
+    <!-- Removing gz_ros2_control plugin to prevent multiple plugin instances causing segfaults -->
   </model>
 </sdf>

File: components/simulations/PicknPlace/robot_config/urdf/ur/ur5/ur_macro.xacro (robot description, xacro)
@@ -60,5 +60,4 @@
     fake_sensor_commands:=false
     sim_gazebo:=false
-    sim_ignition:=false
     headless_mode:=false
     initial_positions:=${dict(shoulder_pan_joint=-1.57,shoulder_lift_joint=-1.57,elbow_joint=0.0,wrist_1_joint=-1.57,wrist_2_joint=0.0,wrist_3_joint=0.0)}
@@ -84,5 +83,5 @@
       physical_parameters_file="${physical_parameters_file}"
       visual_parameters_file="${visual_parameters_file}"
-      force_abs_paths="${sim_gazebo or sim_ignition}"/>
+      force_abs_paths="${sim_gazebo}"/>
     <!-- ros2 control include -->
     <xacro:include filename="$(find robot_config)/urdf/ur/ur5/ur_ros2_control.xacro" />
@@ -95,5 +94,4 @@
       headless_mode="${headless_mode}"
       sim_gazebo="${sim_gazebo}"
-      sim_ignition="${sim_ignition}"
       script_filename="${script_filename}"
       output_recipe_filename="${output_recipe_filename}"
@@ -236,17 +234,5 @@
           <xacro:get_mesh name="wrist_3" type="collision"/>
         </geometry>
-        <surface>
-        <friction>
-          <ode>
-            <mu>100000.0</mu>
-            <mu2>100000.0</mu2>
-          </ode>
-        </friction>
-        <contact>
-          <ode>
-            <min_depth>0.003</min_depth>
-          </ode>
-        </contact>
-      </surface>
+        <!-- Gazebo Classic surface/friction parameters removed - not supported in Harmonic -->
       </collision>
       <xacro:cylinder_inertial radius="${wrist_3_inertia_radius}" length="${wrist_3_inertia_length}"  mass="${wrist_3_mass}">
@@ -359,12 +345,5 @@
           <box size="0.01 0.01 0.01"/>
         </geometry>
-        <surface>
-          <friction>
-            <ode>
-              <mu>10</mu>
-              <mu2>10</mu2>
-            </ode>
-          </friction>
-        </surface>
+        <!-- Gazebo Classic surface/friction parameters removed - not supported in Harmonic -->
         <origin rpy="0 0 0" xyz="-0.01 0 0"/>
       </collision>

File: components/simulations/PicknPlace/robot_config/urdf/ur/ur5/ur_macro_modified.xacro (robot description, xacro)
@@ -60,5 +60,4 @@
     fake_sensor_commands:=false
     sim_gazebo:=false
-    sim_ignition:=false
     headless_mode:=false
     initial_positions:=${dict(shoulder_pan_joint=-1.57,shoulder_lift_joint=-1.57,elbow_joint=0.0,wrist_1_joint=-1.57,wrist_2_joint=0.0,wrist_3_joint=0.0)}
@@ -84,5 +83,5 @@
       physical_parameters_file="${physical_parameters_file}"
       visual_parameters_file="${visual_parameters_file}"
-      force_abs_paths="${sim_gazebo or sim_ignition}"/>
+      force_abs_paths="${sim_gazebo }"/>
     <!-- ros2 control include -->
     <xacro:include filename="$(find robot_config)/urdf/ur/ur5/ur_ros2_control.xacro" />
@@ -95,5 +94,4 @@
       headless_mode="${headless_mode}"
       sim_gazebo="${sim_gazebo}"
-      sim_ignition="${sim_ignition}"
       script_filename="${script_filename}"
       output_recipe_filename="${output_recipe_filename}"

File: components/simulations/PicknPlace/robot_config/urdf/ur/ur5/ur_ros2_control.xacro (robot description, xacro)
@@ -6,5 +6,4 @@
     use_fake_hardware:=false fake_sensor_commands:=false
     sim_gazebo:=false
-    sim_ignition:=false
     headless_mode:=false
     initial_positions:=${dict(shoulder_pan_joint=0.0,shoulder_lift_joint=-1.57,elbow_joint=0.0,wrist_1_joint=-1.57,wrist_2_joint=0.0,wrist_3_joint=0.0)}
@@ -20,8 +19,9 @@
       <hardware>
         <xacro:if value="${sim_gazebo}">
-          <plugin>gazebo_ros2_control/GazeboSystem</plugin>
-        </xacro:if>
-        <xacro:if value="${sim_ignition}">
-          <plugin>ign_ros2_control/IgnitionSystem</plugin>
+          <plugin>gz_ros2_control/GazeboSimSystem</plugin>
+          <!-- position_proportional_gain MUST be inside <hardware> so GazeboSimSystem
+               reads it at initialization. Setting via YAML /** or ros2 param set only
+               reaches the ROS parameter server, not the hardware interface. -->
+          <param name="position_proportional_gain">100.0</param>
         </xacro:if>
         <xacro:if value="${use_fake_hardware}">
@@ -30,5 +30,5 @@
           <param name="state_following_offset">0.0</param>
         </xacro:if>
-        <xacro:unless value="${use_fake_hardware or sim_gazebo or sim_ignition}">
+        <xacro:unless value="${use_fake_hardware or sim_gazebo}">
           <plugin>ur_robot_driver/URPositionHardwareInterface</plugin>
           <param name="robot_ip">${robot_ip}</param>
@@ -57,6 +57,6 @@
       <joint name="${prefix}shoulder_pan_joint">
         <command_interface name="position">
-          <param name="min">{-2*pi}</param>
-          <param name="max">{2*pi}</param>
+          <param name="min">-6.28318</param>
+          <param name="max">6.28318</param>
         </command_interface>
         <command_interface name="velocity">
@@ -73,6 +73,6 @@
       <joint name="${prefix}shoulder_lift_joint">
         <command_interface name="position">
-          <param name="min">{-2*pi}</param>
-          <param name="max">{2*pi}</param>
+          <param name="min">-6.28318</param>
+          <param name="max">6.28318</param>
         </command_interface>
         <command_interface name="velocity">
@@ -89,6 +89,6 @@
       <joint name="${prefix}elbow_joint">
         <command_interface name="position">
-          <param name="min">{-pi}</param>
-          <param name="max">{pi}</param>
+          <param name="min">-3.14159</param>
+          <param name="max">3.14159</param>
         </command_interface>
         <command_interface name="velocity">
@@ -105,6 +105,6 @@
       <joint name="${prefix}wrist_1_joint">
         <command_interface name="position">
-          <param name="min">{-2*pi}</param>
-          <param name="max">{2*pi}</param>
+          <param name="min">-6.28318</param>
+          <param name="max">6.28318</param>
         </command_interface>
         <command_interface name="velocity">
@@ -121,6 +121,6 @@
       <joint name="${prefix}wrist_2_joint">
         <command_interface name="position">
-          <param name="min">{-2*pi}</param>
-          <param name="max">{2*pi}</param>
+          <param name="min">-6.28318</param>
+          <param name="max">6.28318</param>
         </command_interface>
         <command_interface name="velocity">
@@ -137,6 +137,6 @@
       <joint name="${prefix}wrist_3_joint">
         <command_interface name="position">
-          <param name="min">{-2*pi}</param>
-          <param name="max">{2*pi}</param>
+          <param name="min">-6.28318</param>
+          <param name="max">6.28318</param>
         </command_interface>
         <command_interface name="velocity">
@@ -151,15 +151,30 @@
         <state_interface name="effort"/>
       </joint>
-      <joint name="${prefix}gripper_joint1">
-        <command_interface name="position"/>
-        <state_interface name="position">
-        <param name="initial_value">0</param>
-        </state_interface>
-      </joint>
-      <joint name="${prefix}gripper_joint2">
-        <command_interface name="position"/>
-        <state_interface name="position"/>
-      </joint>
-      <xacro:unless value="${sim_gazebo or sim_ignition}">
+      <!-- Gripper finger joints (merged here so they share the same GazeboSimSystem hardware as arm joints) -->
+      <!-- Right finger mirrors left finger via mimic param; both controlled by gripper_controller -->
+      <xacro:if value="${sim_gazebo}">
+        <joint name="${prefix}left_finger_joint">
+          <command_interface name="position">
+            <param name="min">0.0</param>
+            <param name="max">0.035</param>
+          </command_interface>
+          <command_interface name="velocity"/>
+          <state_interface name="position">
+            <param name="initial_value">0.0</param>
+          </state_interface>
+          <state_interface name="velocity"/>
+          <state_interface name="effort"/>
+        </joint>
+        <joint name="${prefix}right_finger_joint">
+          <param name="mimic">${prefix}left_finger_joint</param>
+          <param name="multiplier">1.0</param>
+          <state_interface name="position">
+            <param name="initial_value">0.0</param>
+          </state_interface>
+          <state_interface name="velocity"/>
+          <state_interface name="effort"/>
+        </joint>
+      </xacro:if>
+      <xacro:unless value="${sim_gazebo }">
         <sensor name="tcp_fts_sensor">
           <state_interface name="force.x"/>

File: components/simulations/PicknPlace/robot_config/urdf/ur/ur5/ur_ros2_control_effort.xacro (robot description, xacro)
@@ -6,5 +6,4 @@
     use_fake_hardware:=false fake_sensor_commands:=false
     sim_gazebo:=false
-    sim_ignition:=false
     headless_mode:=false
     initial_positions:=${dict(shoulder_pan_joint=0.0,shoulder_lift_joint=-1.57,elbow_joint=0.0,wrist_1_joint=-1.57,wrist_2_joint=0.0,wrist_3_joint=0.0)}
@@ -20,8 +19,5 @@
       <hardware>
         <xacro:if value="${sim_gazebo}">
-          <plugin>gazebo_ros2_control/GazeboSystem</plugin>
-        </xacro:if>
-        <xacro:if value="${sim_ignition}">
-          <plugin>ign_ros2_control/IgnitionSystem</plugin>
+          <plugin>gz_ros2_control/GazeboSimSystem</plugin>
         </xacro:if>
         <xacro:if value="${use_fake_hardware}">
@@ -30,5 +26,5 @@
           <param name="state_following_offset">0.0</param>
         </xacro:if>
-        <xacro:unless value="${use_fake_hardware or sim_gazebo or sim_ignition}">
+        <xacro:unless value="${use_fake_hardware or sim_gazebo}">
           <plugin>ur_robot_driver/URPositionHardwareInterface</plugin>
           <param name="robot_ip">${robot_ip}</param>
@@ -114,5 +110,5 @@
         <state_interface name="effort"/>
       </joint>
-      <xacro:unless value="${sim_gazebo or sim_ignition}">
+      <xacro:unless value="${sim_gazebo}">
         <sensor name="tcp_fts_sensor">
           <state_interface name="force.x"/>

File: components/simulations/PicknPlace/robot_config/urdf/ur/ur5/ur_urdf.xacro (robot description, xacro)
@@ -38,5 +38,4 @@
    <xacro:arg name="fake_sensor_commands" default="false" />
    <xacro:arg name="sim_gazebo" default="false" />
-   <xacro:arg name="sim_ignition" default="false" />
    <xacro:arg name="simulation_controllers" default="" />
    <!-- initial position for simulations (Fake Hardware, Gazebo, Ignition) -->
@@ -44,6 +43,10 @@
    <xacro:arg name="namespace" default=""/>
    <xacro:arg name="pedestal_height" default=".32"/>
-   <xacro:arg name="vacuum_gripper" default="true"/>
-   <xacro:arg name="finger_gripper" default="false"/>
+   <xacro:arg name="use_gripper" default="true"/>
+   <!-- Spawn position arguments (from launch file) -->
+   <xacro:arg name="spawn_x" default="0.0"/>
+   <xacro:arg name="spawn_y" default="0.0"/>
+   <xacro:arg name="spawn_z" default="0.0"/>
+   <xacro:arg name="spawn_yaw" default="0.0"/>
    <!-- convert to property to use substitution in function -->
    <xacro:property name="initial_positions_file" default="$(arg initial_positions_file)"/>
@@ -66,5 +69,4 @@
      fake_sensor_commands="$(arg fake_sensor_commands)"
      sim_gazebo="$(arg sim_gazebo)"
-     sim_ignition="$(arg sim_ignition)"
      headless_mode="$(arg headless_mode)"
      initial_positions="${xacro.load_yaml(initial_positions_file)}"
@@ -85,4 +87,38 @@
      <origin rpy="0 0 0.0" xyz="0 0 ${$(arg pedestal_height)/2}"/>          <!-- position robot in the world -->
    </xacro:ur_robot>
+   <!-- Pedestal and world joint (always needed for valid URDF tree) -->
+   <link name="$(arg prefix)pedestal">
+     <visual>
+       <origin rpy="0 0 0.0" xyz="0 0 0"/>
+       <geometry>
+         <cylinder radius="0.1" length="$(arg pedestal_height)"/>
+       </geometry>
+       <material name="Grey">
+         <color rgba="0.5 0.5 0.5 1.0"/>
+       </material>
+     </visual>
+     <collision>
+       <origin rpy="0 0 0" xyz="0 0 0.0"/>
+       <geometry>
+         <cylinder radius="0.1" length="$(arg pedestal_height)"/>
+       </geometry>
+     </collision>
+     <inertial>
+       <mass value="120"/>
+       <origin rpy="0 0 0" xyz="0.0 0.0 0.0" />
+       <inertia ixx="100" ixy="0" ixz="0" iyy="120" iyz="0" izz="130"/>
+     </inertial>
+   </link>
+   <joint name="$(arg prefix)world_joint" type="fixed">
+     <parent link="world"/>
+     <child link="$(arg prefix)pedestal"/>
+     <!-- Position pedestal with its center at half-height above ground -->
+     <origin xyz="$(arg spawn_x) $(arg spawn_y) ${$(arg pedestal_height)/2}" rpy="0.0 0.0 $(arg spawn_yaw)"/>
+   </joint>
+   <!-- Include parallel gripper for grasping -->
+   <xacro:if value="$(arg use_gripper)">
+     <xacro:include filename="$(find robot_config)/urdf/ur/ur5/parallel_gripper.xacro" />
+     <xacro:parallel_gripper prefix="$(arg prefix)" />
+   </xacro:if>
    <xacro:if value="$(arg sim_gazebo)">
     <!-- Gazebo plugins -->
@@ -111,29 +147,6 @@
         <origin xyz="0 0 0.0" rpy="0 0 0" />
       </joint>
-      <link name="$(arg prefix)pedestal">
-        <visual>
-          <origin rpy="0 0 0.0" xyz="0 0 0"/>
-          <geometry>
-            <cylinder radius="0.1" length="$(arg pedestal_height)"/>
-          </geometry>
-          <material name="Grey">
-            <color rbga="0.5 0.5 0.5"/>
-          </material>
-        </visual>
-        <collision>
-          <origin rpy="0 0 0" xyz="0 0 0.0"/>
-          <geometry>
-            <cylinder radius="0.1" length="$(arg pedestal_height)"/>
-          </geometry>
-        </collision>
-        <inertial>
-          <mass value="120"/>
-          <origin rpy="0 0 0" xyz="0.0 0.0 0.0" />
-          <inertia ixx="100" ixy="0" ixz="0" iyy="120" iyz="0" izz="130"/>
-        </inertial>
-      </link>
       <gazebo reference="$(arg prefix)pedestal">
-        <mu1>0.2</mu1>
-        <mu2>0.2</mu2>
+        <!-- Gazebo Classic physics parameters mu1/mu2 removed - not supported in Harmonic -->
         <material>
           <ambient>1.00 0.44 0.00 1</ambient>
@@ -142,35 +155,15 @@
         </material>
       </gazebo>
-      <joint name="$(arg prefix)world_joint" type="fixed">
-        <parent link="world"/>
-        <child link="$(arg prefix)pedestal"/>
-        <origin rpy="0.0 0.0 0.0" xyz="0 0 ${$(arg pedestal_height)/2}"/>
-      </joint>
-      <xacro:if value="$(arg vacuum_gripper)">
-        <xacro:include filename="$(find robot_config)/urdf/ur/ur5/ur_vacuum.xacro" />
-      </xacro:if>
+      <!-- Gazebo Harmonic ros2_control plugin configuration -->
       <gazebo>
-        <plugin filename="libgz_ros2_control-system.so" name="gz_ros2_control::GazeboSimROS2ControlPlugin">
+        <plugin filename="gz_ros2_control-system" name="gz_ros2_control::GazeboSimROS2ControlPlugin">
           <ros>
             <namespace>$(arg namespace)</namespace>
           </ros>
           <parameters>$(arg simulation_controllers)</parameters>
-          <controller_manager_node_name>$(arg namespace)controller_manager</controller_manager_node_name>
+          <robot_param>robot_description</robot_param>
+          <robot_param_node>robot_state_publisher</robot_param_node>
         </plugin>
       </gazebo>
-  </xacro:if>
-  <xacro:if value="$(eval arg('sim_gazebo') or arg('sim_ignition'))">
-    <!-- Gazebo plugins -->
-    <gazebo reference="world">
-    </gazebo>
-    <gazebo>
-      <plugin filename="libgz_ros2_control-system.so" name="gz_ros2_control::GazeboSimROS2ControlPlugin">
-        <ros>
-          <namespace>$(arg namespace)</namespace>
-        </ros>
-        <parameters>$(arg simulation_controllers)</parameters>
-        <controller_manager_node_name>$(arg prefix)controller_manager</controller_manager_node_name>
-      </plugin>
-    </gazebo>
   </xacro:if>
 <!-- Future reference code to enable camera on the arm-->
@@ -182,4 +175,5 @@
 -->
 <!--
+Example Gazebo Harmonic camera sensor (pure SDF):
  <gazebo reference="camera_link1">
     <sensor name="robot_camera1" type="camera">

File: components/simulations/PicknPlace/robot_config/urdf/ur/ur5/ur_vacuum.xacro (robot description, xacro)
@@ -19,7 +19,7 @@
       </visual>
       <collision name="vacuum_collision_${index}">
-        <origin rpy="0 0 0" xyz="0 0 0.0025"/>
+        <origin rpy="0 0 0" xyz="0 0 0.015"/>
         <geometry>
-          <cylinder radius="0.01" length="0.005"/>
+          <cylinder radius="0.02" length="0.03"/>
         </geometry>
       </collision>
@@ -38,69 +38,27 @@
       <dynamics damping="0.0" friction="10"/>
     </joint>
-    <!-- Contact sensors dla ARIAC plugin -->
+    <!-- Gazebo properties for vacuum gripper -->
     <gazebo reference="${prefix}vacuum_gripper${index}">
-      <mu1>1.0</mu1>
-      <mu2>1.0</mu2>
-      <minDepth>0.003</minDepth>
+      <mu1>5.0</mu1>
+      <mu2>5.0</mu2>
+      <minDepth>0.0005</minDepth>
       <maxVel>0</maxVel>
-      <kp>1e+13</kp>
-      <kd>1.0</kd>
+      <kp>1e+18</kp>
+      <kd>1000.0</kd>
       <material>Gazebo/Grey</material>
-      <!-- Contact sensor 1 -->
-      <sensor name="vacuum_contact_sensor_1_${index}" type="contact">
-        <contact>
-          <collision>vacuum_collision_${index}</collision>
-        </contact>
-        <update_rate>100</update_rate>
-        <plugin name="contact_sensor_1_plugin_${index}" filename="libgz_ros_contact.so">
-          <ros>
-            <namespace>${namespace}</namespace>
-            <remapping>~/contacts:=vacuum_gripper${index}/contact_sensor_1</remapping>
-          </ros>
-        </plugin>
-      </sensor>
-      <!-- Contact sensor 2 -->
-      <sensor name="vacuum_contact_sensor_2_${index}" type="contact">
-        <contact>
-          <collision>vacuum_collision_${index}</collision>
-        </contact>
-        <update_rate>100</update_rate>
-        <plugin name="contact_sensor_2_plugin_${index}" filename="libgz_ros_contact.so">
-          <ros>
-            <namespace>${namespace}</namespace>
-            <remapping>~/contacts:=vacuum_gripper${index}/contact_sensor_2</remapping>
-          </ros>
-        </plugin>
-      </sensor>
     </gazebo>
-    <!-- ARIAC Vacuum Tool Plugin -->
+    <!-- DetachableJoint Plugin for vacuum gripper -->
     <gazebo>
-      <plugin name="${prefix}vacuum_tool_plugin_${index}" filename="libariac_vacuum_tool_plugin.so">
-        <ros>
-          <namespace>${namespace}</namespace>
-        </ros>
-        <!-- Basic parameters -->
-        <tool_type>2</tool_type> <!-- VacuumTools::VG_2 -->
-        <gripper_base_link>${prefix}vacuum_gripper${index}</gripper_base_link>
-        <!-- Contact sensor topics -->
-        <contact_sensor_1_topic>/${namespace}/vacuum_gripper${index}/contact_sensor_1</contact_sensor_1_topic>
-        <contact_sensor_2_topic>/${namespace}/vacuum_gripper${index}/contact_sensor_2</contact_sensor_2_topic>
-        <!-- Serwisy ROS -->
-        <attach_service>attach_${index}</attach_service>
-        <detach_service>detach_${index}</detach_service>
-        <!-- Parameters malfunctions (optional) -->
-        <malfunction_occurrence>0</malfunction_occurrence>
-        <grasp_occurrence>1</grasp_occurrence>
-        <!-- Joint for lock/unlock -->
-        <lock_joint>${prefix}gripper_joint${index}</lock_joint>
-        <!-- Physical parameters -->
-        <max_force>50.0</max_force>
-        <max_distance>0.1</max_distance>
-        <min_distance>0.01</min_distance>
+      <plugin name="gz::sim::systems::DetachableJoint" filename="libgz-sim-detachable-joint-system.so">
+        <parent_link>${prefix}vacuum_gripper${index}</parent_link>
+        <child_model>cube_0</child_model>
+        <child_link>link</child_link>
+        <topic>/${namespace}/vacuum_gripper/attach_${index}</topic>
+        <suppress_child_warning>true</suppress_child_warning>
       </plugin>
     </gazebo>
 </xacro:macro>
 <!-- Base link dla vacuum gripper -->
-<link name="vacuum_gripper_base">
+<link name="$(arg prefix)vacuum_gripper_base">
   <gravity>0</gravity>
   <visual name="vacuum_visual_base">
@@ -125,7 +83,7 @@
   </collision>
 </link>
-<joint name="vacuum_gripper_base_joint" type="fixed">
-  <parent link="ee_link" />
-  <child link="vacuum_gripper_base" />
+<joint name="$(arg prefix)vacuum_gripper_base_joint" type="fixed">
+  <parent link="$(arg prefix)ee_link" />
+  <child link="$(arg prefix)vacuum_gripper_base" />
   <origin rpy="0.0 0.0 0.0" xyz="0.0025 0.0 0.0"/>
   <limit effort="0.0" velocity="0.0" lower="0" upper="0" />
@@ -133,5 +91,5 @@
 </joint>
 <!-- Gazebo properties dla base -->
-<gazebo reference="vacuum_gripper_base">
+<gazebo reference="$(arg prefix)vacuum_gripper_base">
   <material>Gazebo/DarkGrey</material>
 </gazebo>
@@ -141,5 +99,5 @@
   namespace="$(arg namespace)"
   index="1"
-  base_link="vacuum_gripper_base"
+  base_link="$(arg prefix)vacuum_gripper_base"
   xyz="0.0 0.0125 0.002"/>
 <xacro:ur_vacuum_gripper
@@ -147,5 +105,5 @@
   namespace="$(arg namespace)"
   index="2"
-  base_link="vacuum_gripper_base"
+  base_link="$(arg prefix)vacuum_gripper_base"
   xyz="0.0 -0.0125 0.002"/>
 </robot>
